Commit message: Update my_robot.xacro

File: my_robot/urdf/my_robot.xacro (robot description, xacro)
@@ -180,3 +180,16 @@
     <dynamics damping="1.0" friction="1.0"/>
   </joint>
+<!-- Add color to components -->
+  <gazebo reference="chassis">
+    <material>Gazebo/Orange</material>
+  </gazebo>
+  <gazebo reference="right_wheel">
+    <material>Gazebo/Green</material>
+  </gazebo>
+<gazebo reference="left_wheel">
+    <material>Gazebo/Green</material>
+  </gazebo>
+<gazebo reference="camera">
+    <material>Gazebo/Red</material>
+  </gazebo>
 </robot>

Commit message: Update my_robot.xacro

File: my_robot/urdf/my_robot.xacro (robot description, xacro)
@@ -69,5 +69,5 @@
       <origin xyz="0 0 0" rpy="0 1.5707 1.5707"/>
       <geometry>
-        <cylinder radius="0.1" length="0.05"/>
+        <cylinder radius="0.3" length="0.05"/>
       </geometry>
     </collision>
@@ -75,5 +75,5 @@
       <origin xyz="0 0 0" rpy="0 1.5707 1.5707"/>
       <geometry>
-        <cylinder radius="0.1" length="0.05"/>
+        <cylinder radius="0.3" length="0.05"/>
       </geometry>
     </visual>
@@ -91,5 +91,5 @@
       <origin xyz="0 0 0" rpy="0 1.5707 1.5707"/>
       <geometry>
-        <cylinder radius="0.1" length="0.05"/>
+        <cylinder radius="0.3" length="0.05"/>
       </geometry>
     </collision>
@@ -97,5 +97,5 @@
       <origin xyz="0 0 0" rpy="0 1.5707 1.5707"/>
       <geometry>
-        <cylinder radius="0.1" length="0.05"/>
+        <cylinder radius="0.3" length="0.05"/>
       </geometry>
     </visual>

Commit message: Update my_robot.xacro

File: my_robot/urdf/my_robot.xacro (robot description, xacro)
@@ -69,5 +69,5 @@
       <origin xyz="0 0 0" rpy="0 1.5707 1.5707"/>
       <geometry>
-        <cylinder radius="0.3" length="0.05"/>
+        <cylinder radius="0.15" length="0.05"/>
       </geometry>
     </collision>
@@ -75,5 +75,5 @@
       <origin xyz="0 0 0" rpy="0 1.5707 1.5707"/>
       <geometry>
-        <cylinder radius="0.3" length="0.05"/>
+        <cylinder radius="0.15" length="0.05"/>
       </geometry>
     </visual>
@@ -91,5 +91,5 @@
       <origin xyz="0 0 0" rpy="0 1.5707 1.5707"/>
       <geometry>
-        <cylinder radius="0.3" length="0.05"/>
+        <cylinder radius="0.15" length="0.05"/>
       </geometry>
     </collision>
@@ -97,5 +97,5 @@
       <origin xyz="0 0 0" rpy="0 1.5707 1.5707"/>
       <geometry>
-        <cylinder radius="0.3" length="0.05"/>
+        <cylinder radius="0.15" length="0.05"/>
       </geometry>
     </visual>
@@ -142,5 +142,5 @@
   </link>
   <joint type="fixed" name="camera_joint">
-    <origin xyz="0.2 0.15 0" rpy="0 0 0"/>
+    <origin xyz="0.2 0.0 0" rpy="0 0 0"/>
     <child link="camera"/>
     <parent link="chassis"/>

Commit message: Update my_robot.xacro

File: my_robot/urdf/my_robot.xacro (robot description, xacro)
@@ -22,5 +22,5 @@
       <origin xyz="0 0 0" rpy=" 0 0 0"/>
       <geometry>
-        <box size=".4 .2 .1"/>
+        <box size=".4 .2 .15"/>
       </geometry>
     </collision>
@@ -28,5 +28,5 @@
       <origin xyz="0 0 0" rpy=" 0 0 0"/>
       <geometry>
-        <box size=".4 .2 .1"/>
+        <box size=".4 .2 .15"/>
       </geometry>
     </visual>

Commit message: Update my_robot.xacro

File: my_robot/urdf/my_robot.xacro (robot description, xacro)
@@ -69,5 +69,5 @@
       <origin xyz="0 0 0" rpy="0 1.5707 1.5707"/>
       <geometry>
-        <cylinder radius="0.15" length="0.05"/>
+        <cylinder radius="0.12" length="0.05"/>
       </geometry>
     </collision>
@@ -75,5 +75,5 @@
       <origin xyz="0 0 0" rpy="0 1.5707 1.5707"/>
       <geometry>
-        <cylinder radius="0.15" length="0.05"/>
+        <cylinder radius="0.12" length="0.05"/>
       </geometry>
     </visual>
@@ -91,5 +91,5 @@
       <origin xyz="0 0 0" rpy="0 1.5707 1.5707"/>
       <geometry>
-        <cylinder radius="0.15" length="0.05"/>
+        <cylinder radius="0.12" length="0.05"/>
       </geometry>
     </collision>
@@ -97,5 +97,5 @@
       <origin xyz="0 0 0" rpy="0 1.5707 1.5707"/>
       <geometry>
-        <cylinder radius="0.15" length="0.05"/>
+        <cylinder radius="0.12" length="0.05"/>
       </geometry>
     </visual>

Commit message: Update my_robot.xacro

File: my_robot/urdf/my_robot.xacro (robot description, xacro)
@@ -69,5 +69,5 @@
       <origin xyz="0 0 0" rpy="0 1.5707 1.5707"/>
       <geometry>
-        <cylinder radius="0.12" length="0.05"/>
+        <cylinder radius="0.101" length="0.05"/>
       </geometry>
     </collision>
@@ -75,5 +75,5 @@
       <origin xyz="0 0 0" rpy="0 1.5707 1.5707"/>
       <geometry>
-        <cylinder radius="0.12" length="0.05"/>
+        <cylinder radius="0.101" length="0.05"/>
       </geometry>
     </visual>
@@ -91,5 +91,5 @@
       <origin xyz="0 0 0" rpy="0 1.5707 1.5707"/>
       <geometry>
-        <cylinder radius="0.12" length="0.05"/>
+        <cylinder radius="0.101" length="0.05"/>
       </geometry>
     </collision>
@@ -97,5 +97,5 @@
       <origin xyz="0 0 0" rpy="0 1.5707 1.5707"/>
       <geometry>
-        <cylinder radius="0.12" length="0.05"/>
+        <cylinder radius="0.101" length="0.05"/>
       </geometry>
     </visual>

Commit message: Update my_robot.xacro

File: my_robot/urdf/my_robot.xacro (robot description, xacro)
@@ -69,5 +69,5 @@
       <origin xyz="0 0 0" rpy="0 1.5707 1.5707"/>
       <geometry>
-        <cylinder radius="0.101" length="0.05"/>
+        <cylinder radius="0.05" length="0.05"/>
       </geometry>
     </collision>
@@ -75,5 +75,5 @@
       <origin xyz="0 0 0" rpy="0 1.5707 1.5707"/>
       <geometry>
-        <cylinder radius="0.101" length="0.05"/>
+        <cylinder radius="0.05" length="0.05"/>
       </geometry>
     </visual>
@@ -91,5 +91,5 @@
       <origin xyz="0 0 0" rpy="0 1.5707 1.5707"/>
       <geometry>
-        <cylinder radius="0.101" length="0.05"/>
+        <cylinder radius="0.05" length="0.05"/>
       </geometry>
     </collision>
@@ -97,5 +97,5 @@
       <origin xyz="0 0 0" rpy="0 1.5707 1.5707"/>
       <geometry>
-        <cylinder radius="0.101" length="0.05"/>
+        <cylinder radius="0.05" length="0.05"/>
       </geometry>
     </visual>

Commit message: Update my_robot.xacro

File: my_robot/urdf/my_robot.xacro (robot description, xacro)
@@ -69,5 +69,5 @@
       <origin xyz="0 0 0" rpy="0 1.5707 1.5707"/>
       <geometry>
-        <cylinder radius="0.05" length="0.05"/>
+        <cylinder radius="0.08" length="0.05"/>
       </geometry>
     </collision>
@@ -75,5 +75,5 @@
       <origin xyz="0 0 0" rpy="0 1.5707 1.5707"/>
       <geometry>
-        <cylinder radius="0.05" length="0.05"/>
+        <cylinder radius="0.08" length="0.05"/>
       </geometry>
     </visual>
@@ -91,5 +91,5 @@
       <origin xyz="0 0 0" rpy="0 1.5707 1.5707"/>
       <geometry>
-        <cylinder radius="0.05" length="0.05"/>
+        <cylinder radius="0.08" length="0.05"/>
       </geometry>
     </collision>
@@ -97,5 +97,5 @@
       <origin xyz="0 0 0" rpy="0 1.5707 1.5707"/>
       <geometry>
-        <cylinder radius="0.05" length="0.05"/>
+        <cylinder radius="0.08" length="0.05"/>
       </geometry>
     </visual>

Commit message: Update my_robot.xacro

File: my_robot/urdf/my_robot.xacro (robot description, xacro)
@@ -69,5 +69,5 @@
       <origin xyz="0 0 0" rpy="0 1.5707 1.5707"/>
       <geometry>
-        <cylinder radius="0.08" length="0.05"/>
+        <cylinder radius="0.1001" length="0.05"/>
       </geometry>
     </collision>
@@ -75,5 +75,5 @@
       <origin xyz="0 0 0" rpy="0 1.5707 1.5707"/>
       <geometry>
-        <cylinder radius="0.08" length="0.05"/>
+        <cylinder radius="0.1001" length="0.05"/>
       </geometry>
     </visual>
@@ -91,5 +91,5 @@
       <origin xyz="0 0 0" rpy="0 1.5707 1.5707"/>
       <geometry>
-        <cylinder radius="0.08" length="0.05"/>
+        <cylinder radius="0.1001" length="0.05"/>
       </geometry>
     </collision>
@@ -97,5 +97,5 @@
       <origin xyz="0 0 0" rpy="0 1.5707 1.5707"/>
       <geometry>
-        <cylinder radius="0.08" length="0.05"/>
+        <cylinder radius="0.1001" length="0.05"/>
       </geometry>
     </visual>

Commit message: Update my_robot.xacro

File: my_robot/urdf/my_robot.xacro (robot description, xacro)
@@ -22,5 +22,5 @@
       <origin xyz="0 0 0" rpy=" 0 0 0"/>
       <geometry>
-        <box size=".4 .2 .15"/>
+        <box size=".4 .2 .088"/>
       </geometry>
     </collision>
